File: ECAD/KnokooPedalCtrl/KnokooPedalCtrl.kicad_pcb (KiCad board)
At the start: 2 copper layers, 46.4 x 39.4 mm, 19 parts, among them J1 MAIN PCB CONNECTION, J2 Conn_01x04, J3 UI, J5 ICSP, U2 PIC12F1572

Commit message: v0.1
Small pinout and silkscreen fixes
Connections:
- J2 pad 1: (no net) -> Net-(J2-Pad1)
- J2 pad 2: /KNOKKO_ON -> /Intensity
- J2 pad 4: /Intensity -> /KNOKKO_ON
- J5 pad 6: (no net) -> Net-(J5-Pad6)
Routing:
- net /KNOKKO_ON: track 42.6 -> 50.6 mm
- net /Intensity: track 26.2 -> 24.2 mm, vias 0 -> 1
Other:
- board text added: "KNOK POTI"
- board text added: "SCHILK v0.1 KNOKOO MOD"
- board text added: "VS 0V 5V"
- board text removed: "POTI"
- board text removed: "SCHILK v0.0 KNOKOO MOD"
Changed lines of the file:
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@@
     (thickness 1.6)
     (drawings 17)
-    (tracks 164)
+    (tracks 167)
     (zones 0)
     (modules 19)
-    (nets 13)
+    (nets 15)
   )
   (page A4)
   (title_block
     (title "Knokoo Pedal Mod")
-    (date 2020-09-26)
-    (rev v0.0)
+    (date 2020-10-17)
+    (rev v0.1)
     (company "Philipp Schilk")
   )
@@
       (drillshape 0)
       (scaleselection 1)
-      (outputdirectory "ProductionFiles/Gerber/"))
+      (outputdirectory "../ProductionFiles/Gerber/"))
   )
   (net 0 "")
@@
   (net 11 /LED)
   (net 12 "Net-(J5-Pad1)")
+  (net 13 "Net-(J2-Pad1)")
+  (net 14 "Net-(J5-Pad6)")
   (net_class Default "This is the default net class."
     (clearance 0.2)
@@
     (fp_line (start -2.95 -2.8) (end -2.95 9.7) (layer F.CrtYd) (width 0.05))
     (pad 4 thru_hole oval (at 7.5 0 270) (size 1.7 1.95) (drill 0.95) (layers *.Cu *.Mask)
-      (net 6 /Intensity))
+      (net 7 /KNOKKO_ON))
     (pad 3 thru_hole oval (at 5 0 270) (size 1.7 1.95) (drill 0.95) (layers *.Cu *.Mask)
       (net 1 GND))
     (pad 2 thru_hole oval (at 2.5 0 270) (size 1.7 1.95) (drill 0.95) (layers *.Cu *.Mask)
-      (net 7 /KNOKKO_ON))
-    (pad 1 thru_hole roundrect (at 0 0 270) (size 1.7 1.95) (drill 0.95) (layers *.Cu *.Mask) (roundrect_rratio 0.147059))
+      (net 6 /Intensity))
+    (pad 1 thru_hole roundrect (at 0 0 270) (size 1.7 1.95) (drill 0.95) (layers *.Cu *.Mask) (roundrect_rratio 0.147059)
+      (net 13 "Net-(J2-Pad1)"))
     (model ${KISYS3DMOD}/Connector_JST.3dshapes/JST_XH_S4B-XH-A_1x04_P2.50mm_Horizontal.wrl
       (at (xyz 0 0 0))
@@
     (fp_line (start 1.27 -1.27) (end 1.27 13.97) (layer F.Fab) (width 0.1))
     (fp_line (start -0.635 -1.27) (end 1.27 -1.27) (layer F.Fab) (width 0.1))
-    (pad 6 thru_hole oval (at 0 12.7 90) (size 1.7 1.7) (drill 1) (layers *.Cu *.Mask))
+    (pad 6 thru_hole oval (at 0 12.7 90) (size 1.7 1.7) (drill 1) (layers *.Cu *.Mask)
+      (net 14 "Net-(J5-Pad6)"))
     (pad 5 thru_hole oval (at 0 10.16 90) (size 1.7 1.7) (drill 1) (layers *.Cu *.Mask)
       (net 4 "Net-(D1-Pad2)"))
@@
   (gr_line (start 54.61 57.15) (end 54.61 90.805) (layer Edge.Cuts) (width 0.05))
   (gr_poly (pts (xy 73.66 58.42) (xy 72.39 59.69) (xy 72.39 57.15)) (layer F.SilkS) (width 0.1))
-  (gr_text "SCHILK  v0.0\nKNOKOO MOD " (at 64.77 92.3925) (layer F.SilkS)
+  (gr_text "SCHILK  v0.1\nKNOKOO MOD " (at 64.77 92.3925) (layer F.SilkS)
     (effects (font (size 1.5 1.5) (thickness 0.3)) (justify left))
   )
@@
     (effects (font (size 1.5 1.5) (thickness 0.3)))
   )
-  (gr_text POTI (at 58.1025 86.36) (layer F.SilkS)
+  (gr_text "KNOK POTI" (at 61.595 86.36) (layer F.SilkS)
     (effects (font (size 1.5 1.5) (thickness 0.3)))
   )
@@
     (effects (font (size 1.5 1.5) (thickness 0.3)))
   )
-  (gr_text "5V\n0V\nVS" (at 69.215 62.865) (layer F.SilkS)
+  (gr_text "VS\n0V\n5V\n\n" (at 69.215 64.135) (layer F.SilkS)
     (effects (font (size 1.5 1.5) (thickness 0.3)))
   )
-  (gr_text "PEDC\nPEDP\nPED+\nLED-\nLED+\nPOTs\nPOT-\nPOT+" (at 85.09 83.185) (layer F.SilkS)
-    (effects (font (size 1.45 1.5) (thickness 0.3)))
+  (gr_text "PEDC\nPEDP\nPED+\nLED-\nLED+\nPOTs\nPOT-\nPOT+" (at 81.915 83.185) (layer F.SilkS)
+    (effects (font (size 1.45 1.5) (thickness 0.3)) (justify left))
   )
   (segment (start 64.77 62.825) (end 75.05 62.825) (width 0.5) (layer F.Cu) (net 1))
@@
   (segment (start 63.795 60.325) (end 60.96 63.16) (width 0.25) (layer F.Cu) (net 6))
   (segment (start 64.77 60.325) (end 63.795 60.325) (width 0.25) (layer F.Cu) (net 6))
-  (segment (start 63.545 82.1125) (end 64.77 82.1125) (width 0.25) (layer F.Cu) (net 6))
-  (segment (start 60.96 79.5275) (end 63.545 82.1125) (width 0.25) (layer F.Cu) (net 6))
-  (segment (start 60.96 79.0575) (end 60.96 79.5275) (width 0.25) (layer F.Cu) (net 6))
-  (segment (start 60.96 63.16) (end 60.96 79.0575) (width 0.25) (layer F.Cu) (net 6))
+  (via (at 60.96 78.105) (size 0.8) (drill 0.4) (layers F.Cu B.Cu) (net 6))
+  (segment (start 60.96 63.16) (end 60.96 78.105) (width 0.25) (layer F.Cu) (net 6))
+  (segment (start 63.7775 78.105) (end 64.77 77.1125) (width 0.25) (layer B.Cu) (net 6))
+  (segment (start 60.96 78.105) (end 63.7775 78.105) (width 0.25) (layer B.Cu) (net 6))
   (segment (start 89.47 67.945) (end 87.436768 67.945) (width 0.25) (layer F.Cu) (net 7))
   (segment (start 81.310501 66.130001) (end 80.614499 66.130001) (width 0.25) (layer F.Cu) (net 7))
@@
   (segment (start 82.680494 66.04999) (end 82.580502 65.949998) (width 0.25) (layer F.Cu) (net 7))
   (segment (start 87.436768 67.945) (end 85.541758 66.04999) (width 0.25) (layer F.Cu) (net 7))
-  (segment (start 63.545 77.1125) (end 64.77 77.1125) (width 0.25) (layer F.Cu) (net 7))
-  (segment (start 62.23 75.7975) (end 63.545 77.1125) (width 0.25) (layer F.Cu) (net 7))
-  (segment (start 62.23 75.565) (end 62.23 75.7975) (width 0.25) (layer F.Cu) (net 7))
-  (segment (start 62.23 66.078285) (end 62.23 75.565) (width 0.25) (layer F.Cu) (net 7))
+  (segment (start 62.23 66.078285) (end 62.23 74.295) (width 0.25) (layer F.Cu) (net 7))
+  (segment (start 63.72251 75.78751) (end 66.26251 75.78751) (width 0.25) (layer F.Cu) (net 7))
+  (segment (start 62.23 74.295) (end 63.72251 75.78751) (width 0.25) (layer F.Cu) (net 7))
+  (segment (start 66.26251 75.78751) (end 66.675 76.2) (width 0.25) (layer F.Cu) (net 7))
+  (segment (start 65.995 82.1125) (end 64.77 82.1125) (width 0.25) (layer F.Cu) (net 7))
+  (segment (start 66.675 81.4325) (end 65.995 82.1125) (width 0.25) (layer F.Cu) (net 7))
+  (segment (start 66.675 76.2) (end 66.675 81.4325) (width 0.25) (layer F.Cu) (net 7))
   (segment (start 74.93 72.8725) (end 77.47 72.8725) (width 0.25) (layer F.Cu) (net 8))
   (segment (start 89.58 74.575) (end 88.665 73.66) (width 0.25) (layer B.Cu) (net 8))
@@
       )
     )
+  )
+  (zone (net 0) (net_name "") (layers F&B.Cu) (hatch edge 0.508)
+    (connect_pads (clearance 0.508))
+    (min_thickness 0.254)
+    (keepout (tracks allowed) (vias allowed) (copperpour not_allowed))
+    (fill (arc_segments 32) (thermal_gap 0.508) (thermal_bridge_width 0.508))
+    (polygon
+      (pts
+        (xy 100.965 64.77) (xy 92.075 64.77) (xy 92.075 55.88) (xy 100.965 55.88)
+      )
+    )
+  )
+  (zone (net 0) (net_name "") (layers F&B.Cu) (hatch edge 0.508)
+    (connect_pads (clearance 0.508))
+    (min_thickness 0.254)
+    (keepout (tracks allowed) (vias allowed) (copperpour not_allowed))
+    (fill (arc_segments 32) (thermal_gap 0.508) (thermal_bridge_width 0.508))
+    (polygon
+      (pts
+        (xy 63.5 95.25) (xy 54.61 95.25) (xy 54.61 86.36) (xy 63.5 86.36)
+      )
+    )

Commit message: v0.2
Parts:
- added R6: DNS, Resistor_SMD:R_0603_1608Metric, F.Cu at (81.3, 71.8)
- added R7: DNS, Resistor_SMD:R_0603_1608Metric, F.Cu at (85.1, 71.8)
Connections:
- J2 pad 1: Net-(J2-Pad1) -> (no net)
- J5 pad 6: Net-(J5-Pad6) -> (no net)
Routing:
- net GND: track 63.4 -> 78.1 mm, vias 0 -> 1
- net /Duration_Sense: track 34.3 -> 43.3 mm
- net +5V: track 28.9 -> 34.2 mm
Other:
- board text added: "SCHILK v0.2 KNOKOO MOD"
- board text removed: "5V 0V VS"
- board text removed: "SCHILK v0.1 KNOKOO MOD"
